Commit message: Gazebo Classic 스폰 연동 및 정지 진동/베이스 흔들림 해결
gazebo.launch.py + Gazebo 전용 xacro(gazebo_ros2_control/GazeboSystem)로
스폰~컨트롤러 기동 파이프라인 구성. 정지 시 로봇 전체가 심하게 떨리던
문제를 3중 원인으로 규명 후 해결:

1. 지면 관통: g_base 충돌 메시가 링크 프레임 아래 3cm까지 내려와
   z=0 고정 시 접촉력 vs world 고정조인트 구속 싸움 발생(상시 가진원)
   → world_to_base를 z=0.032로 상향
2. PID D항의 속도 노이즈 증폭 채터링 → kd=0, 감쇠는 URDF
   <dynamics damping>(임계감쇠 기준)으로 이관
3. ODE explicit 감쇠 이산 발산(B > 2·I_local/dt, 국소 관성 작은 J3~J5)
   → 전 관절 implicitSpringDamper 활성화

부가 수정:
- effort_scale arg 신설: inertia_scale과 동일 배율(100) 적용해
  스케일 세계에서 가속 능력 보존 (미적용 시 5 N·m 포화로 J1/J2 수렴 불능)
- controller update_rate 100→1000 Hz (물리 스텝 일치)
- gazebo_ros2_control humble을 ros2.repos에 핀 고정(소스 빌드)

검증: 정지 진동 p2p 0.008° 이하·속도 0, 베이스 원점 오차 <1e-5 m,
6관절 동시 궤적 추종 최대 0.32°, 툴끝 8자 궤적(12cm, IK 161 waypoint) 완주.

Co-Authored-By: Claude Fable 5 <noreply@anthropic.com>

File: src/mycobot_280_lfd_description/urdf/mycobot_280_m5.ros2_control.xacro (robot description, xacro)
@@ -4,15 +4,25 @@
   plugin 인자로 하드웨어 구현을 스왑:
    - 시뮬레이션(현재): mock_components/GenericSystem
-   - Gazebo(W2):       gz_ros2_control/GazeboSimSystem 등
+   - Gazebo(W2):       gazebo_ros2_control/GazeboSystem (use_pid=true 필수)
    - 실기(W7):         pymycobot 기반 자체 hardware_interface
+  use_pid: Gazebo 전용. SetPosition(운동학 강제)은 저관성 체인에서
+  결정론적 한계순환(±17°)을 일으켜 힘 기반 PID(SetForce)로 전환한다.
+  kd=0 고정: Gazebo 속도 신호의 고주파 노이즈가 D항에서 토크로 증폭되어
+  채터링(관절 진동 + 베이스 흔들림)을 유발. 감쇠는 URDF <dynamics damping>
+  (ODE implicit 처리, 임계감쇠 기준)이 담당한다. mock/실기는 pos_* 무시.
 -->
 <robot xmlns:xacro="http://www.ros.org/wiki/xacro">
-  <xacro:macro name="mycobot_280_ros2_control" params="name plugin">
+  <xacro:macro name="mycobot_280_ros2_control" params="name plugin use_pid:=false">
     <ros2_control name="${name}" type="system">
       <hardware>
         <plugin>${plugin}</plugin>
       </hardware>
-      <xacro:macro name="arm_joint" params="joint_name">
+      <xacro:macro name="arm_joint" params="joint_name kp kd ki">
         <joint name="${joint_name}">
+          <xacro:if value="${use_pid}">
+            <param name="pos_kp">${kp}</param>
+            <param name="pos_ki">${ki}</param>
+            <param name="pos_kd">${kd}</param>
+          </xacro:if>
           <command_interface name="position"/>
           <state_interface name="position">
@@ -22,10 +32,13 @@
         </joint>
       </xacro:macro>
-      <xacro:arm_joint joint_name="joint2_to_joint1"/>
-      <xacro:arm_joint joint_name="joint3_to_joint2"/>
-      <xacro:arm_joint joint_name="joint4_to_joint3"/>
-      <xacro:arm_joint joint_name="joint5_to_joint4"/>
-      <xacro:arm_joint joint_name="joint6_to_joint5"/>
-      <xacro:arm_joint joint_name="joint6output_to_joint6"/>
+      <!-- kp는 inertia_scale=100 적용 후 I_eff 기준 (J1,J2≈1.0, J3≈0.3,
+           J4,J5≈0.04, J6≈1e-3 kg·m²), 목표 ω≈5~20rad/s.
+           ζ≈1은 URDF joint damping이 제공 (kd=0 사유는 상단 주석) -->
+      <xacro:arm_joint joint_name="joint2_to_joint1" kp="30.0" kd="0.0" ki="1.0"/>
+      <xacro:arm_joint joint_name="joint3_to_joint2" kp="30.0" kd="0.0" ki="1.0"/>
+      <xacro:arm_joint joint_name="joint4_to_joint3" kp="15.0" kd="0.0" ki="1.0"/>
+      <xacro:arm_joint joint_name="joint5_to_joint4" kp="8.0" kd="0.0" ki="1.0"/>
+      <xacro:arm_joint joint_name="joint6_to_joint5" kp="8.0" kd="0.0" ki="1.0"/>
+      <xacro:arm_joint joint_name="joint6output_to_joint6" kp="2.0" kd="0.0" ki="0.2"/>
     </ros2_control>
   </xacro:macro>

File: src/mycobot_280_lfd_description/urdf/mycobot_280_m5.urdf.xacro (robot description, xacro)
@@ -17,5 +17,14 @@
   <!-- 실기 스펙 관절 최대 속도 120 deg/s -->
   <xacro:property name="joint_vel" value="2.0944"/>
-  <xacro:property name="joint_effort" value="5.0"/>
+  <!-- effort_scale: inertia_scale과 같은 배율로 줘야 스케일된 세계에서
+       가속 능력이 실기와 동일해짐. 미적용 시 PID 출력이 5 N·m에 포화되어
+       kd 큰 관절(J1,J2)이 채터링으로 수렴 불능. mock/실기는 기본 1. -->
+  <xacro:arg name="effort_scale" default="1.0"/>
+  <xacro:property name="joint_effort" value="${5.0*$(arg effort_scale)}"/>
+  <!-- inertia_scale: Gazebo Classic 안정화용 관성 배율 (기본 1 = 실측 근사).
+       질량은 유지(중력 정확)하고 관성 텐서만 키워 저관성 수치 불안정을 회피.
+       위치 제어 궤적 재생에서 운동학 정확도에는 영향 없음. -->
+  <xacro:arg name="inertia_scale" default="1.0"/>
+  <xacro:property name="inertia_scale" value="$(arg inertia_scale)"/>
   <!-- 실린더 근사 관성. axis = 실린더 축 방향(x|y|z), (cx cy cz) = 질량중심 -->
   <xacro:macro name="cyl_inertial" params="mass r h axis cx cy cz">
@@ -23,6 +32,6 @@
       <origin xyz="${cx} ${cy} ${cz}" rpy="0 0 0"/>
       <mass value="${mass}"/>
-      <xacro:property name="i_axial" value="${mass*r*r/2}"/>
-      <xacro:property name="i_trans" value="${mass*(3*r*r+h*h)/12}"/>
+      <xacro:property name="i_axial" value="${inertia_scale*mass*r*r/2}"/>
+      <xacro:property name="i_trans" value="${inertia_scale*mass*(3*r*r+h*h)/12}"/>
       <xacro:if value="${axis == 'x'}">
         <inertia ixx="${i_axial}" ixy="0" ixz="0"
@@ -176,4 +185,12 @@
   </link>
   <!-- ================= 조인트 ================= -->
+  <!-- damping: 임계감쇠 B=2√(kp·I_eff) 기준, inertia_scale에 비례.
+       ODE가 내재적(implicit)으로 처리해 수치 안정 — PID kd로 감쇠를 걸면
+       속도 노이즈가 토크로 증폭돼 채터링/베이스 흔들림을 유발하므로
+       감쇠는 여기서만 담당하고 PID kd=0으로 둔다. -->
+  <xacro:property name="damp_j12" value="${0.11*inertia_scale}"/>
+  <xacro:property name="damp_j3"  value="${0.042*inertia_scale}"/>
+  <xacro:property name="damp_j45" value="${0.011*inertia_scale}"/>
+  <xacro:property name="damp_j6"  value="${0.0009*inertia_scale}"/>
   <joint name="g_base_to_joint1" type="fixed">
     <parent link="g_base"/>
@@ -185,4 +202,5 @@
     <limit effort="${joint_effort}" lower="-2.9321" upper="2.9321"
            velocity="${joint_vel}"/>
+    <dynamics damping="${damp_j12}"/>
     <parent link="joint1"/>
     <child link="joint2"/>
@@ -193,4 +211,5 @@
     <limit effort="${joint_effort}" lower="-2.4434" upper="2.4434"
            velocity="${joint_vel}"/>
+    <dynamics damping="${damp_j12}"/>
     <parent link="joint2"/>
     <child link="joint3"/>
@@ -201,4 +220,5 @@
     <limit effort="${joint_effort}" lower="-2.6179" upper="2.6179"
            velocity="${joint_vel}"/>
+    <dynamics damping="${damp_j3}"/>
     <parent link="joint3"/>
     <child link="joint4"/>
@@ -209,4 +229,5 @@
     <limit effort="${joint_effort}" lower="-2.6179" upper="2.6179"
            velocity="${joint_vel}"/>
+    <dynamics damping="${damp_j45}"/>
     <parent link="joint4"/>
     <child link="joint5"/>
@@ -217,4 +238,5 @@
     <limit effort="${joint_effort}" lower="-2.7052" upper="2.7925"
            velocity="${joint_vel}"/>
+    <dynamics damping="${damp_j45}"/>
     <parent link="joint5"/>
     <child link="joint6"/>
@@ -225,4 +247,5 @@
     <limit effort="${joint_effort}" lower="-3.14159" upper="3.14159"
            velocity="${joint_vel}"/>
+    <dynamics damping="${damp_j6}"/>
     <parent link="joint6"/>
     <child link="joint6_flange"/>
